Commit message: fix the controller and do lqr to calculate full state gains

File: breadcrumb_example/urdf/cartpole.urdf (robot description, URDF)
Before this commit: robot cartpole, 3 links, 2 joints
Joints:
- joint cart_to_world: limit lower=-2.4 upper=2.4 effort=1000 velocity=10 -> lower=-100.0 upper=100.0 effort=1000 velocity=10
